Commit message: feat:增加VLP-16的配置,相应东西还需要优化与确认,现频率太低以及GPU方式出来数据很奇怪

File: description/robot/mbot.xacro (robot description, xacro)
@@ -5,4 +5,5 @@
     <xacro:include filename="$(find robot_gazebo)/description/sensor/imu/imu.xacro" />
     <xacro:include filename="$(find robot_gazebo)/description/sensor/lidar/rplidar/rplidar.xacro" />
+    <xacro:include filename="$(find robot_gazebo)/description/sensor/lidar/velodyne/VLP-16.urdf.xacro" />
     <!--接口说明(函数变量)
         base_radius    车体半径，建议值0.2
@@ -22,14 +23,15 @@
         prefix      sensor_link前缀
         base_length 车体厚度，建议值0.16
-        postion_x   sensor_link底部相对于base平面中心的x方向坐标
-        postion_y   sensor_link底部相对于base平面中心的y方向坐标
-        postion_z   sensor_link底部相对于base平面中心的z方向坐标，亦为sensor_link长度,建议值大于0，0会报错
+        position_x   sensor_link底部相对于base平面中心的x方向坐标
+        position_y   sensor_link底部相对于base平面中心的y方向坐标
+        position_z   sensor_link底部相对于base平面中心的z方向坐标，亦为sensor_link长度,建议值大于0，0会报错
         接口说明(缺省变量)
         sensor_link_radius sensor_link的半径，建议值0.01
     -->
-    <sensor_link prefix="imu"  base_length="0.0" postion_x="0.0" postion_y="0" postion_z="0.001"/>
-    <sensor_link prefix="laser"  base_length="0.16" postion_x="0.1" postion_y="0" postion_z="0.05"/>
+    <sensor_link prefix="imu"  base_length="0.0" position_x="0.0" position_y="0" position_z="0.001"/>
+    <!-- <sensor_link prefix="laser"  base_length="0.16" position_x="0.1" position_y="0" position_z="0.05"/> -->
+    <sensor_link prefix="velodyne"  base_length="0.16" position_x="0.1" position_y="0" position_z="1.0"/>
     <!--接口说明(函数变量)
-        postion_z   laser底部相对于base平面中心的z方向坐标，建议值大于0，0会报错
+        position_z   laser底部相对于base平面中心的z方向坐标，建议值大于0，0会报错
         rotation_r  laser底部相对于base平面中心的roll
         rotation_p  laser底部相对于base平面中心的pitch
@@ -46,5 +48,13 @@
         noise_sttdev      激光数据的高斯噪声方差，建议0.01
     -->
-    <xacro:imu postion_z="0.001" rotation_r="0" rotation_p="0" rotation_y="0" />
-    <xacro:rplidar postion_z="0.05" rotation_r="0" rotation_p="0" rotation_y="0" />
+    <xacro:imu position_z="0.001" rotation_r="0" rotation_p="0" rotation_y="0" />
+    <!-- <xacro:rplidar position_z="0.05" rotation_r="0" rotation_p="0" rotation_y="0" /> -->
+    <!-- here z must be half of position_z-->
+    <xacro:arg name="gpu" default="false"/>
+    <xacro:property name="gpu" value="$(arg gpu)" />
+    <xacro:arg name="organize_cloud" default="false"/>
+    <xacro:property name="organize_cloud" value="$(arg organize_cloud)" />
+    <xacro:VLP-16 parent="velodyne_link" name="velodyne" topic="/velodyne_points" organize_cloud="${organize_cloud}" hz="10" samples="1800" gpu="${gpu}">
+        <origin xyz="0 0 0.5" rpy="0 0 0" />
+    </xacro:VLP-16>
 </robot>

File: description/sensor/imu/imu.xacro (robot description, xacro)
@@ -1,5 +1,5 @@
 <?xml version="1.0"?>
 <robot name="imu" xmlns:xacro="http://www.ros.org/wiki/xacro">
-    <xacro:macro name="imu" params="postion_z
+    <xacro:macro name="imu" params="position_z
                                     rotation_r
                                     rotation_p
@@ -38,7 +38,7 @@
                 <update_rate>10</update_rate>
                 <visualize>true</visualize>
-                <topic>/imu/data</topic>
+                <topic>/imu</topic>
                 <plugin filename="libgazebo_ros_imu_sensor.so" name="imu_plugin">
-                    <topicName>imu/data</topicName>
+                    <topicName>imu</topicName>
                     <bodyName>base_link</bodyName>
                     <updateRateHZ>100.0</updateRateHZ>

File: description/sensor/lidar/rplidar/rplidar.xacro (robot description, xacro)
@@ -12,5 +12,5 @@
     <xacro:property name="noise_sttdev" value="0.01"/>
     <!--接口说明(函数变量)
-        postion_z   laser底部相对于base平面中心的z方向坐标，建议值大于0，0会报错
+        position_z   laser底部相对于base平面中心的z方向坐标，建议值大于0，0会报错
         rotation_r  laser底部相对于base平面中心的roll
         rotation_p  laser底部相对于base平面中心的pitch
@@ -28,14 +28,14 @@
         一般需要修改获取到的传感器文件几处地方，parent_link,joint的origin和rpy，传感器插件变量
     -->
-    <xacro:macro name="rplidar" params="postion_z
+    <xacro:macro name="rplidar" params="position_z
                                         rotation_r
                                         rotation_p
                                         rotation_y ">
         <joint name="laser_joint" type="fixed">
-            <origin xyz="0 0 ${postion_z/2+laser_length/2}" rpy="${rotation_r} ${rotation_p} ${rotation_y}" />
+            <origin xyz="0 0 ${position_z/2+laser_length/2}" rpy="${rotation_r} ${rotation_p} ${rotation_y}" />
             <parent link="laser_link"/>
-            <child link="laser"/>
+            <child link="base_scan"/>
         </joint>
-        <link name="laser">
+        <link name="base_scan">
             <inertial>
                 <mass value="0.01" />
@@ -58,8 +58,8 @@
             </collision>
         </link>
-        <gazebo reference="laser">
+        <gazebo reference="base_scan">
             <material>Gazebo/Black</material>
         </gazebo>
-        <gazebo reference="laser">
+        <gazebo reference="base_scan">
             <sensor type="ray" name="rplidar">
                 <pose>0 0 0 0 0 0</pose>
@@ -88,5 +88,5 @@
                 <plugin name="gazebo_rplidar" filename="libgazebo_ros_laser.so">
                     <topicName>/scan</topicName>
-                    <frameName>laser</frameName>
+                    <frameName>base_scan</frameName>
                 </plugin>
             </sensor>

File: description/sensor/sensor_link/sensor_link.xacro (robot description, xacro)
@@ -5,7 +5,7 @@
         prefix      sensor_link前缀
         base_length 车体厚度，建议值0.16
-        postion_x   sensor_link底部相对于base平面中心的x方向坐标
-        postion_y   sensor_link底部相对于base平面中心的y方向坐标
-        postion_z   sensor_link底部相对于base平面中心的z方向坐标，亦为sensor_link长度,建议值大于0，0会报错
+        position_x   sensor_link底部相对于base平面中心的x方向坐标
+        position_y   sensor_link底部相对于base平面中心的y方向坐标
+        position_z   sensor_link底部相对于base平面中心的z方向坐标，亦为sensor_link长度,建议值大于0，0会报错
         接口说明(缺省变量)
         sensor_link_radius sensor_link的半径，建议值0.01
@@ -13,9 +13,9 @@
     <xacro:macro name="sensor_link" params="prefix
                                             base_length
-                                            postion_x
-                                            postion_y
-                                            postion_z  ">
+                                            position_x
+                                            position_y
+                                            position_z  ">
         <joint name="${prefix}_link_joint" type="fixed">
-            <origin xyz="${postion_x} ${postion_y} ${base_length/2+postion_z/2}" rpy="0 0 0" />
+            <origin xyz="${position_x} ${position_y} ${base_length/2+position_z/2}" rpy="0 0 0" />
             <parent link="base_link"/>
             <child link="${prefix}_link"/>
@@ -32,5 +32,5 @@
                 <origin xyz=" 0 0 0 " rpy="0 0 0" />
                 <geometry>
-                    <cylinder length="${postion_z}" radius="${sensor_link_radius}"/>
+                    <cylinder length="${position_z}" radius="${sensor_link_radius}"/>
                 </geometry>
             </visual>
@@ -38,5 +38,5 @@
                 <origin xyz="0.0 0.0 0.0" rpy="0 0 0" />
                 <geometry>
-                    <cylinder length="${postion_z}" radius="${sensor_link_radius}"/>
+                    <cylinder length="${position_z}" radius="${sensor_link_radius}"/>
                 </geometry>
             </collision>
